File: 2K Keypad.kicad_sch (KiCad schematic)
At the start: 1 part

Commit message: v1 of  schematic and pcb
Parts:
- added C1, C2, C3: 0.1uF, Capacitor_SMD:C_0805_2012Metric, symbol Device:C_Small
- added C4, C5: 22pF, Capacitor_SMD:C_0805_2012Metric, symbol Device:C_Small
- added C6: 10uF, Capacitor_SMD:C_0805_2012Metric, symbol Device:C_Small
- added C7: 1uF, Capacitor_SMD:C_0805_2012Metric, symbol Device:C_Small
- added D1, D2: D_Small, Diode_SMD:D_SOD-123, symbol Device:D_Small
- added F1: Polyfuse_Small, Fuse:Fuse_1206_3216Metric, symbol Device:Polyfuse_Small
- added MX1, MX2: MX-NoLED, MX_Only:MXOnly-1U-NoLED, symbol MX_Alps_Hybrid:MX-NoLED
- added P1: USB_C_Plug_USB2.0, Connector_USB:USB_C_Receptacle_GCT_USB4085, symbol Connector:USB_C_Plug_USB2.0
- added R1, R2: 22, Resistor_SMD:R_0805_2012Metric, symbol Device:R_Small
- added R3, R4: 10k, Resistor_SMD:R_0805_2012Metric, symbol Device:R_Small
- added R5, R6: 5.1k, Resistor_SMD:R_0805_2012Metric, symbol Device:R_Small
- added SW1: SW_Push, random-keyboard-parts:SKQG-1155865, symbol Switch:SW_Push
- added Y1: 16MHz, Crystal:Crystal_SMD_3225-4Pin_3.2x2.5mm, symbol Device:Crystal_GND24_Small
- gave numbers to parts that had none: 1
Connections:
- net +5V: now also U1.7 (VBUS), C1.1, C2.1, C3.1, C6.1, F1.2, R3.1
- net GND: now also C1.2, C2.2, C3.2, C4.1, C5.1, C6.2, C7.2, P1.A1 (GND), P1.A12 (GND), P1.B1 (GND), P1.B12 (GND), P1.S1 (SHIELD), R4.2, R5.2, R6.2, SW1.1, Y1.2, Y1.4
- net at U1.13 (~{RESET}): now also R3.2, SW1.2
- net at U1.16 (XTAL2): now also C5.2, Y1.3
- net at U1.17 (XTAL1): now also C4.2, Y1.1
- net Row 0: now reaches U1.27 (PD7)
- net Row 0: now also D1.1 (K), D2.1 (K)
- net Col 1: now reaches U1.28 (PB4)
- net Col 1: now also MX2.1 (COL)
- net Col 0: now reaches U1.29 (PB5)
- net Col 0: now also MX1.1 (COL)
- net at U1.3 (D-): now also R1.2
- net at U1.33 (~{HWB}/PE2): now also R4.1
- net at U1.4 (D+): now also R2.1
- net at U1.6 (UCAP): now also C7.1
- new net: P1.A5 (CC), R6.1
- new net: D1.2 (A), MX1.2 (ROW)
- new net: P1.B5 (VCONN), R5.1
- new net: D2.2 (A), MX2.2 (ROW)
- new net D+: P1.A6 (D+), R2.2
- new net D-: P1.A7 (D-), R1.1
- new net VCC: F1.1, P1.A4 (VBUS), P1.A9 (VBUS), P1.B4 (VBUS), P1.B9 (VBUS)
